Commit message: New world created, change in the chasing logic, changed the color of the robot

File: Project2_Chase_it/catkin_ws/src/my_robot/urdf/my_robot.xacro (robot description, xacro)
@@ -177,15 +177,16 @@
     <parent link="chassis"/>
   </joint>
+  <!-- Assign colors to parts of the robot -->
   <gazebo reference="left_wheel">
-    <material>Gazebo/Green</material>
+    <material>Gazebo/ZincYellow</material>
   </gazebo>
   <gazebo reference="right_wheel">
-    <material>Gazebo/Green</material>
+    <material>Gazebo/ZincYellow</material>
   </gazebo>
   <gazebo reference="chassis">
-    <material>Gazebo/Blue</material>
+    <material>Gazebo/Turquoise</material>
   </gazebo>
   <gazebo reference="camera">
-    <material>Gazebo/Red</material>
+    <material>Gazebo/SkyBlue</material>
   </gazebo>
 </robot>

Commit message: Change robot geometry

File: Project2_Chase_it/catkin_ws/src/my_robot/urdf/my_robot.xacro (robot description, xacro)
@@ -8,12 +8,12 @@
   </joint>
   <link name='chassis'>
-    <pose>0 0 0.1 0 0 0</pose>
+    <pose>0 0 0.15 0 0 0</pose>
     <inertial>
-      <mass value="15.0"/>
+      <mass value="50.0"/>
       <origin xyz="0.0 0 0" rpy=" 0 0 0"/>
       <inertia
-          ixx="0.1" ixy="0" ixz="0"
-          iyy="0.1" iyz="0"
-          izz="0.1"
+          ixx="0.3375" ixy="0" ixz="0"
+          iyy="0.3375" iyz="0"
+          izz="0.3375"
       />
     </inertial>
@@ -21,5 +21,5 @@
       <origin xyz="0 0 0" rpy=" 0 0 0"/>
       <geometry>
-        <box size=".4 .2 .1"/>
+        <box size=".6 .3 .15"/>
       </geometry>
     </collision>
@@ -27,29 +27,29 @@
       <origin xyz="0 0 0" rpy=" 0 0 0"/>
       <geometry>
-        <box size=".4 .2 .1"/>
+        <box size=".6 .3 .15"/>
       </geometry>
     </visual>
     <collision name='back_caster_collision'>
-      <origin xyz="-0.15 0 -0.05" rpy=" 0 0 0"/>
+      <origin xyz="-0.225 0 -0.075" rpy=" 0 0 0"/>
       <geometry>
-        <sphere radius="0.0499"/>
+        <sphere radius="0.07485"/>
       </geometry>
     </collision>
     <visual name='back_caster_visual'>
-      <origin xyz="-0.15 0 -0.05" rpy=" 0 0 0"/>
+      <origin xyz="-0.225 0 -0.075" rpy=" 0 0 0"/>
       <geometry>
-        <sphere radius="0.05"/>
+        <sphere radius="0.075"/>
       </geometry>
     </visual>
     <collision name='front_caster_collision'>
-      <origin xyz="0.15 0 -0.05" rpy=" 0 0 0"/>
+      <origin xyz="0.225 0 -0.075" rpy=" 0 0 0"/>
       <geometry>
-        <sphere radius="0.0499"/>
+        <sphere radius="0.07485"/>
       </geometry>
     </collision>
     <visual name='front_caster_visual'>
-      <origin xyz="0.15 0 -0.05" rpy=" 0 0 0"/>
+      <origin xyz="0.225 0 -0.075" rpy=" 0 0 0"/>
       <geometry>
-        <sphere radius="0.05"/>
+        <sphere radius="0.075"/>
       </geometry>
     </visual>
@@ -58,15 +58,15 @@
   <link name='left_wheel'>
    <inertial>
-      <mass value="5.0"/>
+      <mass value="17.0"/>
       <origin xyz="0.0 0.0 0.0" rpy="0.0 1.5707 1.5707"/>
       <inertia
-          ixx="0.1" ixy="0" ixz="0"
-          iyy="0.1" iyz="0"
-          izz="0.1"/>
+          ixx="0.3375" ixy="0" ixz="0"
+          iyy="0.3375" iyz="0"
+          izz="0.3375"/>
     </inertial>
     <collision>
       <origin xyz="0.0 0.0 0.0" rpy="0.0 1.5707 1.5707"/>
       <geometry>
-        <cylinder length="0.05" radius="0.1"/>
+        <cylinder length="0.075" radius="0.15"/>
       </geometry>
     </collision>
@@ -74,5 +74,5 @@
       <origin xyz="0.0 0.0 0.0" rpy="0.0 1.5707 1.5707"/>
       <geometry>
-        <cylinder length="0.05" radius="0.1"/>
+        <cylinder length="0.075" radius="0.15"/>
       </geometry>
     </visual>
@@ -81,15 +81,15 @@
   <link name='right_wheel'>
    <inertial>
-      <mass value="5.0"/>
+      <mass value="15.0"/>
       <origin xyz="0.0 0.0 0.0" rpy="0.0 1.5707 1.5707"/>
       <inertia
-          ixx="0.1" ixy="0" ixz="0"
-          iyy="0.1" iyz="0"
-          izz="0.1"/>
+          ixx="0.3375" ixy="0" ixz="0"
+          iyy="0.3375" iyz="0"
+          izz="0.3375"/>
     </inertial>
     <collision>
       <origin xyz="0.0 0.0 0.0" rpy="0.0 1.5707 1.5707"/>
       <geometry>
-        <cylinder length="0.05" radius="0.1"/>
+        <cylinder length="0.075" radius="0.15"/>
       </geometry>
     </collision>
@@ -97,5 +97,5 @@
       <origin xyz="0.0 0.0 0.0" rpy="0.0 1.5707 1.5707"/>
       <geometry>
-        <cylinder length="0.05" radius="0.1"/>
+        <cylinder length="0.075" radius="0.15"/>
       </geometry>
     </visual>
@@ -103,5 +103,5 @@
   <!-- Wheel joints -->
   <joint type="continuous" name="left_wheel_hinge">
-    <origin xyz="0 0.15 0" rpy="0 0 0"/>
+    <origin xyz="0 0.225 0" rpy="0 0 0"/>
     <child link="left_wheel"/>
     <parent link="chassis"/>
@@ -111,5 +111,5 @@
   </joint>
   <joint type="continuous" name="right_wheel_hinge">
-    <origin xyz="0 -0.15 0" rpy="0 0 0"/>
+    <origin xyz="0 -0.225 0" rpy="0 0 0"/>
     <child link="right_wheel"/>
     <parent link="chassis"/>
@@ -144,5 +144,5 @@
   <joint name="camera_joint" type="fixed">
     <axis xyz="0 1 0" rpy="0 0 0"/>
-    <origin xyz="0.2 0.0 0" rpy="0 0 0"/>
+    <origin xyz="0.3 0.0 0" rpy="0 0 0"/>
     <child link="camera"/>
     <parent link="chassis"/>
@@ -173,5 +173,5 @@
   <joint name="hokuyo_joint" type="fixed">
     <axis xyz="0 1 0" rpy="0 0 0"/>
-    <origin xyz="0.15 0.0 0.1" rpy="0 0 0"/>
+    <origin xyz="0.225 0.0 0.15" rpy="0 0 0"/>
     <child link="hokuyo"/>
     <parent link="chassis"/>
