Commit message: Respond to review comments

File: Project3_Where_am_I/catkin_ws/src/my_robot/urdf/my_robot.xacro (robot description, xacro)
@@ -3,5 +3,5 @@
   <link name="robot_footprint"></link>
   <joint name="robot_footprint_joint" type="fixed">
-    <origin xyz="0 0 0" rpy="0 0 0" />
+    <origin xyz="0 0 0.15" rpy="0 0 0" />
     <parent link="robot_footprint"/>
     <child link="chassis" />
