Commit message: Project4: WIP

File: Project4_Map_my_world/catkin_ws/src/my_robot/urdf/my_robot.xacro (robot description, xacro)
@@ -148,4 +148,12 @@
     <parent link="chassis"/>
   </joint>
+  <!-- Depth camera -->
+  <joint name="camera_optical_joint" type="fixed">
+    <origin xyz="0 0 0" rpy="-1.5707 0 -1.5707"/>
+    <parent link="camera"/>
+    <child link="camera_link_optical"/>
+  </joint>
+  <link name="camera_link_optical">
+  </link>
   <!-- Lidar -->
   <link name="hokuyo">
